File: pcb/AudioSwitch.kicad_pcb (KiCad board)
At the start: 2 copper layers, 100 x 37 mm, 11 parts, among them J1 IN_L, J2 IN_R, J3 OUT1_L, J4 OUT1_R, J5 OUT2_L, J6 OUT2_R, SW1 MRB22B

Commit message: style: add tear drops and rounded tracks
Routing:
- net /OUT1_S: track 8.55 -> 10.1 mm
- net /OUT2_S: track 8.55 -> 10.1 mm
- net /IN_S: track 8.55 -> 10.1 mm
- net /IN_L: track 39.7 -> 39.1 mm
- net /IN_R: track 59.0 -> 58.4 mm
